Commit message: Fixed urdf files

File: urdf/Abstract_env.urdf (robot description, URDF)
Before this commit: robot Abstract_env, 1 links, 0 joints
Links:
- link base_link: geometry collision mesh filename=package://hpp-ompl-benchmark/mesh/Abstract_env.stl; visual mesh filename=package://hpp-ompl-benchmark/mesh/Abstract_env.stl

File: urdf/Abstract_robot.urdf (robot description, URDF)
Before this commit: robot Abstract_robot, 1 links, 0 joints
Links:
- link base_link: geometry collision mesh filename=package://hpp-ompl-benchmark/mesh/Abstract_robot.stl; visual mesh filename=package://hpp-ompl-benchmark/mesh/Abstract_robot.stl

File: urdf/cubicles_env.urdf (robot description, URDF)
Before this commit: robot cubicles_env, 1 links, 0 joints
Links:
- link base_link: geometry collision mesh filename=package://hpp-ompl-benchmark/mesh/cubicles_env.stl; visual mesh filename=package://hpp-ompl-benchmark/mesh/cubicles_env.stl

File: urdf/cubicles_robot.urdf (robot description, URDF)
Before this commit: robot cubicles_robot, 1 links, 0 joints
Links:
- link base_link: geometry collision mesh filename=package://hpp-ompl-benchmark/mesh/cubicles_robot.stl; visual mesh filename=package://hpp-ompl-benchmark/mesh/cubicles_robot.stl

File: urdf/pipedream_env.urdf (robot description, URDF)
Before this commit: robot pipedream_env, 1 links, 0 joints
Links:
- link base_link: geometry collision mesh filename=package://hpp-ompl-benchmark/mesh/pipedream_env.stl; visual mesh filename=package://hpp-ompl-benchmark/mesh/pipedream_env.stl

File: urdf/ring.urdf (robot description, URDF)
Before this commit: robot ring, 1 links, 0 joints
Links:
- link base_link: geometry collision mesh filename=package://hpp-ompl-benchmark/mesh/ring.stl; visual mesh filename=package://hpp-ompl-benchmark/mesh/ring.stl
