Commit message: correct meshs for cubicles and adjust configurations parameters

File: urdf/cubicles_env.urdf (robot description, URDF)
Before this commit: robot cubicles_env, 1 links, 0 joints
Links:
- link base_link: geometry collision mesh filename=package://hpp-ompl-benchmark/mesh/cubicles_envBIG.stl; visual mesh filename=package://hpp-ompl-benchmark/mesh/cubicles_envBIG.stl

File: urdf/cubicles_robot.urdf (robot description, URDF)
Before this commit: robot cubicles_robot, 1 links, 0 joints
Links:
- link base_link: geometry collision mesh filename=package://hpp-ompl-benchmark/mesh/cubicles_robotCENTER.stl; visual mesh filename=package://hpp-ompl-benchmark/mesh/cubicles_robotCENTER.stl
